File: starfire-core.sch (EAGLE design)
At the start: 68 parts, among them Q1 FDN340P, Y1 16MHZ

Commit message: starfire eaglecad lbr refernce moved.
I renamed and moved the EagleCAD library for the PCB fab compoment to our public git repo.  So updated the BRD and SCH references so that users can find the correct library.
Parts:
- FAB: device CircuitMonkey-solaris:PCB-4-MTG-BASE-B1 -> solstice-design-system:PCB-4-MTG-BASE-B1
Changed lines of the file:
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@@
 <part name="SUPPLY62" library="supply2" deviceset="VCC" device=""/>
 <part name="SUPPLY63" library="supply2" deviceset="VCC" device=""/>
-<part name="FAB" library="CircuitMonkey-solaris" deviceset="PCB-4-MTG" device="-BASE-B1" value="STARFIRE PCB"/>
+<part name="FAB" library="solstice-design-system" deviceset="PCB-4-MTG" device="-BASE-B1" value="STARFIRE PCB"/>
 <part name="SUPPLY58" library="supply2" deviceset="GND" device=""/>
 <part name="SUPPLY59" library="supply2" deviceset="GND" device=""/>

Commit message: Rev. A PCBs shared to world
Parts:
- removed WS1, WS10, WS11, WS12, WS13, WS14, WS15, WS16, WS2, WS3, WS4, WS5, WS6, WS7, WS8, WS9: WS2812, led:NEOPPIXEL5X5
- added C17, C18: 10uf, Seeed-Capacitor:CERAMIC-10UF-10V-10%-X5R(0603)
- added SK0, SK1, SK10, SK11, SK12, SK13, SK14, SK15, SK2, SK3, SK4, SK5, SK6, SK7, SK8, SK9: SK6812-MINI, led:SK6812MINI
- added UMBRA: DF12-20DS-0.5V, co-hirose:DF12-20P-RCPT
- added US0, US1, US2: TPSMD-040-RND, con-testpoints:TPSMD-040-RND
- RESET: value B3U-1000P-2P-SMD -> MOM (OFF)-ON; device Seeed-Switch:SMD-BUTTON(2P-3.0X2.5X1.2+0.4MM)-B3U-1000P-2P-SMD -> comp-switch:TACTILE-2PSMD
- VR33: value XC6206P332MR-G-SOT23 -> 3.3V
Connections:
- removed net MOSI/WS2812: ICSP.5, R8.1, UC.PB2
- removed net N$29: WS11.IN, WS12.OUT
- removed net N$30: WS12.IN, WS13.OUT
- removed net N$31: WS13.IN, WS14.OUT
- removed net N$32: WS14.IN, WS15.OUT
- removed net N$33: WS15.IN, WS16.OUT
- removed net PIXELS: R8.2, WS1.OUT
- removed net SCK: ICSP.2, UC.PB1
- new net MOSI: ICSP.5, UC.PB2, UMBRA.16
- new net N$1: SK0.OUT, SK1.IN
- new net N$12: SK6.OUT, SK7.IN
- new net N$4: SK1.OUT, SK2.IN
- new net N$5: SK2.OUT, SK3.IN
- new net N$6: SK3.OUT, SK4.IN
- new net N$9: SK4.OUT, SK5.IN
- new net SCK/PIXELS: ICSP.2, R8.1, UC.PB1, UMBRA.12
- new net SL0: UMBRA.2, US0.P$1
- new net SL1: UMBRA.4, US1.P$1
- new net SL2: UMBRA.6, US2.P$1
- net !RESET: now also RESET.1, UMBRA.10; no longer RESET.2
- net +3V3: now also UMBRA.8
- net D0: now also UMBRA.15
- net D1: now also UMBRA.13
- net D2: now also UMBRA.11
- net D3: now also UMBRA.9
- net D4: now also UMBRA.7
- net D5: now also UMBRA.5
- net D6: now also UMBRA.3
- net D7: now also UMBRA.1
- net GND: now also C17.1, C18.1, HL4.1, RESET.2, SK0.GND, SK1.GND, SK10.GND, SK11.GND, SK12.GND, SK13.GND, SK14.GND, SK15.GND, SK2.GND, SK3.GND, SK4.GND, SK5.GND, SK6.GND, SK7.GND, SK8.GND, SK9.GND, UMBRA.19, UMBRA.20; no longer HL4.2, RESET.1, WS1.GND, WS10.GND, WS11.GND, WS12.GND, WS13.GND, WS14.GND, WS15.GND, WS16.GND, WS2.GND, WS3.GND, WS4.GND, WS5.GND, WS6.GND, WS7.GND, WS8.GND, WS9.GND
- net MISO: now also UMBRA.14
- net N$11: now also SK5.OUT, SK6.IN; no longer WS1.IN, WS2.OUT
- net N$13: now also SK8.OUT, SK9.IN; no longer WS2.IN, WS3.OUT
- net N$14: now also R8.2, SK0.IN; no longer WS3.IN, WS4.OUT
- net N$15: now also SK10.IN, SK9.OUT; no longer WS4.IN, WS5.OUT
- net N$16: now also SK10.OUT, SK11.IN; no longer WS5.IN, WS6.OUT
- net N$17: now also SK11.OUT, SK12.IN; no longer WS6.IN, WS7.OUT
- net N$18: now also SK12.OUT, SK13.IN; no longer WS7.IN, WS8.OUT
- net N$19: now also SK13.OUT, SK14.IN; no longer WS8.IN, WS9.OUT
- net N$20: now also SK14.OUT, SK15.IN; no longer WS10.OUT, WS9.IN
- net N$28: now also SK7.OUT, SK8.IN; no longer WS10.IN, WS11.OUT
- net VCC: now also C17.2, C18.2, SK0.VDD, SK1.VDD, SK10.VDD, SK11.VDD, SK12.VDD, SK13.VDD, SK14.VDD, SK15.VDD, SK2.VDD, SK3.VDD, SK4.VDD, SK5.VDD, SK6.VDD, SK7.VDD, SK8.VDD, SK9.VDD, UMBRA.17, UMBRA.18; no longer WS1.VDD, WS10.VDD, WS11.VDD, WS12.VDD, WS13.VDD, WS14.VDD, WS15.VDD, WS16.VDD, WS2.VDD, WS3.VDD, WS4.VDD, WS5.VDD, WS6.VDD, WS7.VDD, WS8.VDD, WS9.VDD
- net VIN: now also HL4.2; no longer HL4.1
Other:
- moved on the sheet: D13, R3, R4, R5, R8

Commit message: Revision B released
Added Umbra connector feature along with Umbra mount support holes.  RGB LEDs are now smaller SK6812 type 3.5x3.5mm.   Added output test points for external LED chain that extends on-board chain.  Added PIXEL_EN solder jumper so that user can disable on board pixels if needed.
Parts:
- added EN_PIXELS: (no value), rlc:SOLDER_JUMPER-80MIL-RND
- added PXGND, PXO: TPSMD-040-RND, con-testpoints:TPSMD-040-RND
- added R2: 330R, Seeed-Resistor:SMD-RES-330R-1%-1/10W(0603)
- USB: value ZX62-B-5PA -> USB-Micro-SMT+THD
Connections:
- new net N$29: PXO.P$1, R2.1
- new net N$30: R2.2, SK15.OUT
- new net PIXELS: EN_PIXELS.P$2, R8.1
- net +3V3: now also OPAMPA.-IN2; no longer OPAMPG$1.-IN2
- net D13: now also OPAMPB.+IN1; no longer OPAMPG$2.+IN1
- net GND: now also OPAMPB.GND, PXGND.P$1; no longer OPAMPG$2.GND
- net N$34: now also OPAMPB.-IN1, OPAMPB.OUT1; no longer OPAMPG$2.-IN1, OPAMPG$2.OUT1
- net N$35: now also OPAMPA.OUT2; no longer OPAMPG$1.OUT2
- net SCK/PIXELS: now also EN_PIXELS.P$1; no longer R8.1
- net VCC: now also OPAMPB.+V; no longer OPAMPG$2.+V
- net VCTL: now also OPAMPA.+IN2; no longer OPAMPG$1.+IN2
